File: esp32-beacon-receiver/esp32-beacon-receiver.kicad_sch (KiCad schematic)
At the start: 67 parts, among them J1 USB_B_Micro, J2 Micro_SD_Card, J3 Neopixel, J4 Conn_02x05_Odd_Even, M1 Motor_Servo, Q1 Q_PMOS_GSD, Q2 Q_PMOS_GSD, Q3 MMBT3904, Q4 MMBT3904, U1 PCF8563T, U2 CH340C, U3 ESP32-WROOM-32, U4 TPS54331, U5 FP6291, U6 MAX98357, U7 Logo, Y1 Crystal

Commit message: Fixed some things
Parts:
- removed J4: Conn_02x05_Odd_Even, Connector_PinHeader_2.54mm:PinHeader_2x06_P2.54mm_Vertical, symbol Connector_Generic:Conn_02x06_Odd_Even
- removed TP1: TestPoint, Connector_PinHeader_2.54mm:PinHeader_1x01_P2.54mm_Vertical, symbol Connector:TestPoint
- removed U3: ESP32-WROOM-32, cacophony-footprints:ESP32-WROOM-32, symbol RF_Module:ESP32-WROOM-32
- removed U5: FP6291, Package_TO_SOT_SMD:SOT-23-6, symbol cacophony-symbols:FP6291
- added C20: 47pF, Capacitor_SMD:C_0402_1005Metric, symbol Device:C_Small
- added C21, C23: 10nF, Capacitor_SMD:C_0402_1005Metric, symbol Device:C_Small
- added C22, C24, C25, C30, C31: 22uF, Capacitor_SMD:C_0805_2012Metric, symbol Device:C_Small
- added C26, C29: 1uF, Capacitor_SMD:C_0402_1005Metric, symbol Device:C_Small
- added C27: 100nF, Capacitor_SMD:C_0402_1005Metric, symbol Device:C_Small
- added C28: 10uF, Capacitor_SMD:C_0603_1608Metric, symbol Device:C_Small
- added J4, J5: Conn_01x03, Connector_PinSocket_2.54mm:PinSocket_1x03_P2.54mm_Vertical, symbol Connector_Generic:Conn_01x03
- added R18: 10K, Resistor_SMD:R_0402_1005Metric, symbol Device:R
- added SW2: SW_Push, Button_Switch_SMD:SW_SPST_SKQG_WithStem, symbol Switch:SW_Push
- added U3: ESP32-WROOM-32, cacophony-footprints:ESP32-WROOM-32, symbol cacophony-symbols:ESP32-WROOM-32
- added U5: TPS54331, Package_SO:SOIC-8-1EP_3.9x4.9mm_P1.27mm_EP2.29x3mm, symbol cacophony-symbols:TPS54331
- C1, C6, C9: value 100nF -> 1uF; LCSC C307331 -> C52923
- C10, C15: value 22uF -> 4.7uF; footprint Capacitor_SMD:C_0805_2012Metric -> Capacitor_SMD:C_0402_1005Metric; LCSC C45783 -> C23733
- C12: value 100nF -> 1nF; LCSC C307331 -> C1523
- C16, C17: value 47uF -> 22uF; LCSC C16780 -> C45783
- J2: footprint cacophony-footprints:microSD_HC_Molex_104031-0811 -> cacophony-footprints:SD_Micro
- L2: value 3.3uH -> 6.8uH; footprint Inductor_SMD:L_Sunlord_MWSA0518_5.4x5.2mm -> cacophony-footprints:SWPA5040S; LCSC C408409 -> C36411
- R11: value 68K -> 12K; LCSC C36871 -> C25744
- R15: value 22K -> 2.2K; LCSC C25768 -> C11457
- R7: value 10K -> 100K; LCSC C25744 -> C25741
- R8: value 12K -> 29.4k; LCSC C25752 -> C25890
- U7: footprint cacophony-footprints:logo_small -> cacophony-footprints:logo
Connections:
- net +3V3: now also C9.1, C22.1, C24.1, C25.1, C26.1, U3.2 (VDD)
- net +5V: now also L2.2, R11.1, C29.1, C30.1, C31.1, J4.1 (Pin_1), J5.1 (Pin_1); no longer C10.1, C9.1, D6.1 (K), R15.2
- net BATTERY_VOLTAGE: now also U3.6 (IO34)
- net BUZZER: now also U3.26 (IO4)
- net EN: now also C28.1, SW2.2, U3.3 (EN); no longer C12.1
- net GND: now also D6.2 (A), R15.2, C20.2, C21.2, C22.2, C23.2, C24.2, C25.2, C26.2, C28.2, C29.2, C30.2, C31.2, J4.3 (Pin_3), J5.3 (Pin_3), SW2.1, U3.1 (GND), U3.15 (GND), U3.38 (GND), U3.39 (GND), U5.7 (GND), U5.9 (GND); no longer C12.2, R7.2, U6.4 (SD_MODE)
- net Neopixel: now also U3.12 (IO27)
- net RXD0: now also U3.34 (RXD0/IO3)
- net SCL: now also U3.33 (IO21)
- net SDA: now also U3.36 (IO22)
- net SD_ENABLE: now also U3.28 (IO17)
- net SERVO: now also R18.1, U3.8 (IO32); no longer M1.1 (PWM)
- net STATUS_LED: now also U3.27 (IO16)
- net TXD0: now also U3.35 (TXD0/IO1)
- net VCC: now also C10.1, R7.1, C21.1, U5.2 (VIN); no longer C6.1, L2.1, R1.1
- net at J2.4 (VDD), Q1.3 (D): now also C6.1
- net GAIN: now reaches U6.2 (GAIN_SLOT)
- net GAIN: now also J4.2 (Pin_2)
- net at R11.2, R15.1: now also U5.5 (VSENSE)
- net at R8.1: now also C12.2; no longer R11.1
- net BCLK renamed I2S_BCLK
- net I2S_BCLK: now also U3.10 (IO25)
- net CS renamed SD_CS
- net SD_CS: now also U3.29 (IO5)
- net DIN renamed I2S_DOUT
- net I2S_DOUT: now also U3.9 (IO33)
- net IO0 renamed BOOT_MODE
- net BOOT_MODE: now also U3.25 (IO0)
- net LRCLK renamed I2S_LRCLK
- net I2S_LRCLK: now also U3.11 (IO26)
- net MISO renamed SD_MISO
- net SD_MISO: now also U3.31 (IO19)
- net MOSI renamed SD_MOSI
- net SD_MOSI: now also U3.37 (IO23)
- net RTC_INT# renamed ~{RTC_INT}
- net ~{RTC_INT}: now also U3.7 (IO35)
- net SCK renamed SD_SCK
- net SD_SCK: now also U3.30 (IO18)
- new net: C27.2, D6.1 (K), L2.1, U5.8 (PH)
- new net: C27.1, U5.1 (BOOT)
- new net: C23.1, U5.4 (SS)
- new net: C12.1, C20.1, U5.6 (COMP)
- new net: R1.1, R7.2
- new net: M1.1 (PWM), R18.2
- new net 5V_ENABLE: U3.24 (IO2), U5.3 (EN)
- new net IO12/TDI: U3.14 (IO12)
- new net IO13TCK: U3.16 (IO13)
- new net IO14/TMS: U3.13 (IO14)
- new net IO15/TDO: U3.23 (IO15)
- new net SD_MODE: J5.2 (Pin_2), U6.4 (SD_MODE)
- no-connect marks 20 -> 24
Other:
- moved on the sheet: BZ1, C11, C13, C14, C16, C17, C18, C19, C2, C3, C4, C5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
